Commit message: Add foothold checker node and related configurations
- Updated package.xml to include dependencies for tf2_ros and visualization_msgs.
- Added foothold_checker_node to setup.py for execution.
- Enhanced control_stack.yaml with parameters for foothold checking.
- Integrated foothold_checker_node into control stack launch file.
- Modified view_camera.launch.py to prefer camera-specific RViz config.
- Updated quadruped URDF model with new leg dimensions.
- Created .gitattributes for consistent line endings.
- Implemented foothold_checker_node with depth image processing and foothold evaluation logic.
- Added servo_test.py for testing servo angles using PCA9685.

File: ros2_ws/src/quadruped_description/urdf/quadruped.urdf.xacro (robot description, xacro)
@@ -4,7 +4,7 @@
   <xacro:property name="base_width" value="0.16"/>
   <xacro:property name="base_height" value="0.06"/>
-  <xacro:property name="coxa_length" value="0.05162"/>
-  <xacro:property name="femur_length" value="0.130"/>
-  <xacro:property name="tibia_length" value="0.150"/>
+  <xacro:property name="coxa_length" value="0.035563"/>
+  <xacro:property name="femur_length" value="0.127063"/>
+  <xacro:property name="tibia_length" value="0.127183"/>
   <xacro:property name="link_radius" value="0.012"/>
   <xacro:property name="foot_radius" value="0.018"/>
