Commit message: Switch to final robot model and add bringup tooling

File: ros2_ws/src/Argos_description/urdf/Argos.xacro (robot description, xacro)
@@ -1,7 +1,7 @@
 <?xml version="1.0" ?>
 <robot name="Argos" xmlns:xacro="http://www.ros.org/wiki/xacro">
-<xacro:include filename="$(find Argos_description)/urdf/materials.xacro" />
-<xacro:include filename="$(find Argos_description)/urdf/Argos.trans" />
-<xacro:include filename="$(find Argos_description)/urdf/Argos.gazebo" />
+<xacro:include filename="$(find argos_description)/urdf/materials.xacro" />
+<xacro:include filename="$(find argos_description)/urdf/Argos.trans" />
+<xacro:include filename="$(find argos_description)/urdf/Argos.gazebo" />
 <link name="base_link">
   <inertial>
@@ -13,5 +13,5 @@
     <origin xyz="0 0 0" rpy="0 0 0"/>
     <geometry>
-      <mesh filename="package://Argos_description/meshes/base_link.stl" scale="0.001 0.001 0.001"/>
+      <mesh filename="package://argos_description/meshes/base_link.stl" scale="0.001 0.001 0.001"/>
     </geometry>
     <material name="silver"/>
@@ -20,5 +20,5 @@
     <origin xyz="0 0 0" rpy="0 0 0"/>
     <geometry>
-      <mesh filename="package://Argos_description/meshes/base_link.stl" scale="0.001 0.001 0.001"/>
+      <mesh filename="package://argos_description/meshes/base_link.stl" scale="0.001 0.001 0.001"/>
     </geometry>
   </collision>
@@ -33,5 +33,5 @@
     <origin xyz="-0.009817 0.040183 0.016117" rpy="0 0 0"/>
     <geometry>
-      <mesh filename="package://Argos_description/meshes/chassis_side_left_1.stl" scale="0.001 0.001 0.001"/>
+      <mesh filename="package://argos_description/meshes/chassis_side_left_1.stl" scale="0.001 0.001 0.001"/>
     </geometry>
     <material name="silver"/>
@@ -40,5 +40,5 @@
     <origin xyz="-0.009817 0.040183 0.016117" rpy="0 0 0"/>
     <geometry>
-      <mesh filename="package://Argos_description/meshes/chassis_side_left_1.stl" scale="0.001 0.001 0.001"/>
+      <mesh filename="package://argos_description/meshes/chassis_side_left_1.stl" scale="0.001 0.001 0.001"/>
     </geometry>
   </collision>
@@ -53,5 +53,5 @@
     <origin xyz="0.098183 0.071183 0.016117" rpy="0 0 0"/>
     <geometry>
-      <mesh filename="package://Argos_description/meshes/chassis_front_1.stl" scale="0.001 0.001 0.001"/>
+      <mesh filename="package://argos_description/meshes/chassis_front_1.stl" scale="0.001 0.001 0.001"/>
     </geometry>
     <material name="silver"/>
@@ -60,5 +60,5 @@
     <origin xyz="0.098183 0.071183 0.016117" rpy="0 0 0"/>
     <geometry>
-      <mesh filename="package://Argos_description/meshes/chassis_front_1.stl" scale="0.001 0.001 0.001"/>
+      <mesh filename="package://argos_description/meshes/chassis_front_1.stl" scale="0.001 0.001 0.001"/>
     </geometry>
   </collision>
@@ -73,5 +73,5 @@
     <origin xyz="0.084683 0.031683 0.016117" rpy="0 0 0"/>
     <geometry>
-      <mesh filename="package://Argos_description/meshes/chassis_cam_mount_1.stl" scale="0.001 0.001 0.001"/>
+      <mesh filename="package://argos_description/meshes/chassis_cam_mount_1.stl" scale="0.001 0.001 0.001"/>
     </geometry>
     <material name="silver"/>
@@ -80,5 +80,5 @@
     <origin xyz="0.084683 0.031683 0.016117" rpy="0 0 0"/>
     <geometry>
-      <mesh filename="package://Argos_description/meshes/chassis_cam_mount_1.stl" scale="0.001 0.001 0.001"/>
+      <mesh filename="package://argos_description/meshes/chassis_cam_mount_1.stl" scale="0.001 0.001 0.001"/>
     </geometry>
   </collision>
@@ -93,5 +93,5 @@
     <origin xyz="0.084683 -0.013317 0.016117" rpy="0 0 0"/>
     <geometry>
-      <mesh filename="package://Argos_description/meshes/chassis_cam_mount_2.stl" scale="0.001 0.001 0.001"/>
+      <mesh filename="package://argos_description/meshes/chassis_cam_mount_2.stl" scale="0.001 0.001 0.001"/>
     </geometry>
     <material name="silver"/>
@@ -100,5 +100,5 @@
     <origin xyz="0.084683 -0.013317 0.016117" rpy="0 0 0"/>
     <geometry>
-      <mesh filename="package://Argos_description/meshes/chassis_cam_mount_2.stl" scale="0.001 0.001 0.001"/>
+      <mesh filename="package://argos_description/meshes/chassis_cam_mount_2.stl" scale="0.001 0.001 0.001"/>
     </geometry>
   </collision>
@@ -113,5 +113,5 @@
     <origin xyz="-0.057317 0.009183 0.017617" rpy="0 0 0"/>
     <geometry>
-      <mesh filename="package://Argos_description/meshes/chassis_bottom_1.stl" scale="0.001 0.001 0.001"/>
+      <mesh filename="package://argos_description/meshes/chassis_bottom_1.stl" scale="0.001 0.001 0.001"/>
     </geometry>
     <material name="silver"/>
@@ -120,5 +120,5 @@
     <origin xyz="-0.057317 0.009183 0.017617" rpy="0 0 0"/>
     <geometry>
-      <mesh filename="package://Argos_description/meshes/chassis_bottom_1.stl" scale="0.001 0.001 0.001"/>
+      <mesh filename="package://argos_description/meshes/chassis_bottom_1.stl" scale="0.001 0.001 0.001"/>
     </geometry>
   </collision>
@@ -133,5 +133,5 @@
     <origin xyz="-0.009817 -0.021817 0.016117" rpy="0 0 0"/>
     <geometry>
-      <mesh filename="package://Argos_description/meshes/chassis_side_right__1__1.stl" scale="0.001 0.001 0.001"/>
+      <mesh filename="package://argos_description/meshes/chassis_side_right__1__1.stl" scale="0.001 0.001 0.001"/>
     </geometry>
     <material name="silver"/>
@@ -140,5 +140,5 @@
     <origin xyz="-0.009817 -0.021817 0.016117" rpy="0 0 0"/>
     <geometry>
-      <mesh filename="package://Argos_description/meshes/chassis_side_right__1__1.stl" scale="0.001 0.001 0.001"/>
+      <mesh filename="package://argos_description/meshes/chassis_side_right__1__1.stl" scale="0.001 0.001 0.001"/>
     </geometry>
   </collision>
@@ -153,5 +153,5 @@
     <origin xyz="0.084683 0.031683 -0.022883" rpy="0 0 0"/>
     <geometry>
-      <mesh filename="package://Argos_description/meshes/camera_link_1.stl" scale="0.001 0.001 0.001"/>
+      <mesh filename="package://argos_description/meshes/camera_link_1.stl" scale="0.001 0.001 0.001"/>
     </geometry>
     <material name="silver"/>
@@ -160,25 +160,5 @@
     <origin xyz="0.084683 0.031683 -0.022883" rpy="0 0 0"/>
     <geometry>
-      <mesh filename="package://Argos_description/meshes/camera_link_1.stl" scale="0.001 0.001 0.001"/>
-    </geometry>
-  </collision>
-</link>
-<link name="chassis_top_front_1">
-  <inertial>
-    <origin xyz="0.08406453366502363 0.06199985628852129 0.0014998529519978099" rpy="0 0 0"/>
-    <mass value="0.41722982746680565"/>
-    <inertia ixx="0.000465" iyy="0.001147" izz="0.001612" ixy="0.0" iyz="0.0" ixz="-0.0"/>
-  </inertial>
-  <visual>
-    <origin xyz="0.106183 0.071183 -0.044883" rpy="0 0 0"/>
-    <geometry>
-      <mesh filename="package://Argos_description/meshes/chassis_top_front_1.stl" scale="0.001 0.001 0.001"/>
-    </geometry>
-    <material name="silver"/>
-  </visual>
-  <collision>
-    <origin xyz="0.106183 0.071183 -0.044883" rpy="0 0 0"/>
-    <geometry>
-      <mesh filename="package://Argos_description/meshes/chassis_top_front_1.stl" scale="0.001 0.001 0.001"/>
+      <mesh filename="package://argos_description/meshes/camera_link_1.stl" scale="0.001 0.001 0.001"/>
     </geometry>
   </collision>
@@ -193,5 +173,5 @@
     <origin xyz="-0.220817 -0.052817 0.016117" rpy="0 0 0"/>
     <geometry>
-      <mesh filename="package://Argos_description/meshes/chassis_back_1.stl" scale="0.001 0.001 0.001"/>
+      <mesh filename="package://argos_description/meshes/chassis_back_1.stl" scale="0.001 0.001 0.001"/>
     </geometry>
     <material name="silver"/>
@@ -200,5 +180,5 @@
     <origin xyz="-0.220817 -0.052817 0.016117" rpy="0 0 0"/>
     <geometry>
-      <mesh filename="package://Argos_description/meshes/chassis_back_1.stl" scale="0.001 0.001 0.001"/>
+      <mesh filename="package://argos_description/meshes/chassis_back_1.stl" scale="0.001 0.001 0.001"/>
     </geometry>
   </collision>
@@ -213,5 +193,5 @@
     <origin xyz="-0.220817 -0.052817 -0.044883" rpy="0 0 0"/>
     <geometry>
-      <mesh filename="package://Argos_description/meshes/chassis_top_back_1.stl" scale="0.001 0.001 0.001"/>
+      <mesh filename="package://argos_description/meshes/chassis_top_back_1.stl" scale="0.001 0.001 0.001"/>
     </geometry>
     <material name="silver"/>
@@ -220,5 +200,45 @@
     <origin xyz="-0.220817 -0.052817 -0.044883" rpy="0 0 0"/>
     <geometry>
-      <mesh filename="package://Argos_description/meshes/chassis_top_back_1.stl" scale="0.001 0.001 0.001"/>
+      <mesh filename="package://argos_description/meshes/chassis_top_back_1.stl" scale="0.001 0.001 0.001"/>
+    </geometry>
+  </collision>
+</link>
+<link name="chassis_top_front_1">
+  <inertial>
+    <origin xyz="0.08410298001571184 -0.061989721998729076 0.0014998529519977405" rpy="0 0 0"/>
+    <mass value="0.4159347286719098"/>
+    <inertia ixx="0.000464" iyy="0.001144" izz="0.001607" ixy="0.0" iyz="0.0" ixz="0.0"/>
+  </inertial>
+  <visual>
+    <origin xyz="0.106183 -0.052817 -0.044883" rpy="0 0 0"/>
+    <geometry>
+      <mesh filename="package://argos_description/meshes/chassis_top_front_1.stl" scale="0.001 0.001 0.001"/>
+    </geometry>
+    <material name="silver"/>
+  </visual>
+  <collision>
+    <origin xyz="0.106183 -0.052817 -0.044883" rpy="0 0 0"/>
+    <geometry>
+      <mesh filename="package://argos_description/meshes/chassis_top_front_1.stl" scale="0.001 0.001 0.001"/>
+    </geometry>
+  </collision>
+</link>
+<link name="lidar_link_1">
+  <inertial>
+    <origin xyz="0.033784169392077075 -0.027505085866451538 0.03503813199409616" rpy="0 0 0"/>
+    <mass value="1.122500385833242"/>
+    <inertia ixx="0.000458" iyy="0.000732" izz="0.000909" ixy="-3e-06" iyz="-6e-06" ixz="0.000104"/>
+  </inertial>
+  <visual>
+    <origin xyz="0.079183 -0.018817 -0.047883" rpy="0 0 0"/>
+    <geometry>
+      <mesh filename="package://argos_description/meshes/lidar_link_1.stl" scale="0.001 0.001 0.001"/>
+    </geometry>
+    <material name="silver"/>
+  </visual>
+  <collision>
+    <origin xyz="0.079183 -0.018817 -0.047883" rpy="0 0 0"/>
+    <geometry>
+      <mesh filename="package://argos_description/meshes/lidar_link_1.stl" scale="0.001 0.001 0.001"/>
     </geometry>
   </collision>
@@ -233,5 +253,5 @@
     <origin xyz="0.016983 0.073583 -0.014583" rpy="0 0 0"/>
     <geometry>
-      <mesh filename="package://Argos_description/meshes/FL_coxa_link_1.stl" scale="0.001 0.001 0.001"/>
+      <mesh filename="package://argos_description/meshes/FL_coxa_link_1.stl" scale="0.001 0.001 0.001"/>
     </geometry>
     <material name="silver"/>
@@ -240,5 +260,5 @@
     <origin xyz="0.016983 0.073583 -0.014583" rpy="0 0 0"/>
     <geometry>
-      <mesh filename="package://Argos_description/meshes/FL_coxa_link_1.stl" scale="0.001 0.001 0.001"/>
+      <mesh filename="package://argos_description/meshes/FL_coxa_link_1.stl" scale="0.001 0.001 0.001"/>
     </geometry>
   </collision>
@@ -253,5 +273,5 @@
     <origin xyz="0.041083 0.111383 -0.027133" rpy="0 0 0"/>
     <geometry>
-      <mesh filename="package://Argos_description/meshes/FL_femur_link_1.stl" scale="0.001 0.001 0.001"/>
+      <mesh filename="package://argos_description/meshes/FL_femur_link_1.stl" scale="0.001 0.001 0.001"/>
     </geometry>
     <material name="silver"/>
@@ -260,5 +280,5 @@
     <origin xyz="0.041083 0.111383 -0.027133" rpy="0 0 0"/>
     <geometry>
-      <mesh filename="package://Argos_description/meshes/FL_femur_link_1.stl" scale="0.001 0.001 0.001"/>
+      <mesh filename="package://argos_description/meshes/FL_femur_link_1.stl" scale="0.001 0.001 0.001"/>
     </geometry>
   </collision>
@@ -273,5 +293,5 @@
     <origin xyz="-0.064863 0.110742 0.042899" rpy="0 0 0"/>
     <geometry>
-      <mesh filename="package://Argos_description/meshes/FL_tibia_link_1.stl" scale="0.001 0.001 0.001"/>
+      <mesh filename="package://argos_description/meshes/FL_tibia_link_1.stl" scale="0.001 0.001 0.001"/>
     </geometry>
     <material name="silver"/>
@@ -280,5 +300,5 @@
     <origin xyz="-0.064863 0.110742 0.042899" rpy="0 0 0"/>
     <geometry>
-      <mesh filename="package://Argos_description/meshes/FL_tibia_link_1.stl" scale="0.001 0.001 0.001"/>
+      <mesh filename="package://argos_description/meshes/FL_tibia_link_1.stl" scale="0.001 0.001 0.001"/>
     </geometry>
   </collision>
@@ -293,5 +313,5 @@
     <origin xyz="0.016983 -0.055217 -0.014583" rpy="0 0 0"/>
     <geometry>
-      <mesh filename="package://Argos_description/meshes/FR_coxa_link_1.stl" scale="0.001 0.001 0.001"/>
+      <mesh filename="package://argos_description/meshes/FR_coxa_link_1.stl" scale="0.001 0.001 0.001"/>
     </geometry>
     <material name="silver"/>
@@ -300,5 +320,5 @@
     <origin xyz="0.016983 -0.055217 -0.014583" rpy="0 0 0"/>
     <geometry>
-      <mesh filename="package://Argos_description/meshes/FR_coxa_link_1.stl" scale="0.001 0.001 0.001"/>
+      <mesh filename="package://argos_description/meshes/FR_coxa_link_1.stl" scale="0.001 0.001 0.001"/>
     </geometry>
   </collision>
@@ -313,5 +333,5 @@
     <origin xyz="0.041083 -0.093017 -0.027133" rpy="0 0 0"/>
     <geometry>
-      <mesh filename="package://Argos_description/meshes/FR_femur_link_1.stl" scale="0.001 0.001 0.001"/>
+      <mesh filename="package://argos_description/meshes/FR_femur_link_1.stl" scale="0.001 0.001 0.001"/>
     </geometry>
     <material name="silver"/>
@@ -320,5 +340,5 @@
     <origin xyz="0.041083 -0.093017 -0.027133" rpy="0 0 0"/>
     <geometry>
-      <mesh filename="package://Argos_description/meshes/FR_femur_link_1.stl" scale="0.001 0.001 0.001"/>
+      <mesh filename="package://argos_description/meshes/FR_femur_link_1.stl" scale="0.001 0.001 0.001"/>
     </geometry>
   </collision>
@@ -333,5 +353,5 @@
     <origin xyz="-0.064849 -0.092376 0.04292" rpy="0 0 0"/>
     <geometry>
-      <mesh filename="package://Argos_description/meshes/FR_tibia_link_1.stl" scale="0.001 0.001 0.001"/>
+      <mesh filename="package://argos_description/meshes/FR_tibia_link_1.stl" scale="0.001 0.001 0.001"/>
     </geometry>
     <material name="silver"/>
@@ -340,5 +360,5 @@
     <origin xyz="-0.064849 -0.092376 0.04292" rpy="0 0 0"/>
     <geometry>
-      <mesh filename="package://Argos_description/meshes/FR_tibia_link_1.stl" scale="0.001 0.001 0.001"/>
+      <mesh filename="package://argos_description/meshes/FR_tibia_link_1.stl" scale="0.001 0.001 0.001"/>
     </geometry>
   </collision>
@@ -353,5 +373,5 @@
     <origin xyz="-0.131617 -0.055217 -0.014583" rpy="0 0 0"/>
     <geometry>
-      <mesh filename="package://Argos_description/meshes/RR_coxa_link_1.stl" scale="0.001 0.001 0.001"/>
+      <mesh filename="package://argos_description/meshes/RR_coxa_link_1.stl" scale="0.001 0.001 0.001"/>
     </geometry>
     <material name="silver"/>
@@ -360,5 +380,5 @@
     <origin xyz="-0.131617 -0.055217 -0.014583" rpy="0 0 0"/>
     <geometry>
-      <mesh filename="package://Argos_description/meshes/RR_coxa_link_1.stl" scale="0.001 0.001 0.001"/>
+      <mesh filename="package://argos_description/meshes/RR_coxa_link_1.stl" scale="0.001 0.001 0.001"/>
     </geometry>
   </collision>
@@ -373,5 +393,5 @@
     <origin xyz="-0.176517 -0.093017 -0.027133" rpy="0 0 0"/>
     <geometry>
-      <mesh filename="package://Argos_description/meshes/RR_femur_link_1.stl" scale="0.001 0.001 0.001"/>
+      <mesh filename="package://argos_description/meshes/RR_femur_link_1.stl" scale="0.001 0.001 0.001"/>
     </geometry>
     <material name="silver"/>
@@ -380,5 +400,5 @@
     <origin xyz="-0.176517 -0.093017 -0.027133" rpy="0 0 0"/>
     <geometry>
-      <mesh filename="package://Argos_description/meshes/RR_femur_link_1.stl" scale="0.001 0.001 0.001"/>
+      <mesh filename="package://argos_description/meshes/RR_femur_link_1.stl" scale="0.001 0.001 0.001"/>
     </geometry>
   </collision>
@@ -393,5 +413,5 @@
     <origin xyz="-0.275421 -0.092376 0.052535" rpy="0 0 0"/>
     <geometry>
-      <mesh filename="package://Argos_description/meshes/RR_tibia_link_1.stl" scale="0.001 0.001 0.001"/>
+      <mesh filename="package://argos_description/meshes/RR_tibia_link_1.stl" scale="0.001 0.001 0.001"/>
     </geometry>
     <material name="silver"/>
@@ -400,5 +420,5 @@
     <origin xyz="-0.275421 -0.092376 0.052535" rpy="0 0 0"/>
     <geometry>
-      <mesh filename="package://Argos_description/meshes/RR_tibia_link_1.stl" scale="0.001 0.001 0.001"/>
+      <mesh filename="package://argos_description/meshes/RR_tibia_link_1.stl" scale="0.001 0.001 0.001"/>
     </geometry>
   </collision>
@@ -413,5 +433,5 @@
     <origin xyz="-0.131617 0.073583 -0.014583" rpy="0 0 0"/>
     <geometry>
-      <mesh filename="package://Argos_description/meshes/RL_coxa_link_1.stl" scale="0.001 0.001 0.001"/>
+      <mesh filename="package://argos_description/meshes/RL_coxa_link_1.stl" scale="0.001 0.001 0.001"/>
     </geometry>
     <material name="silver"/>
@@ -420,5 +440,5 @@
     <origin xyz="-0.131617 0.073583 -0.014583" rpy="0 0 0"/>
     <geometry>
-      <mesh filename="package://Argos_description/meshes/RL_coxa_link_1.stl" scale="0.001 0.001 0.001"/>
+      <mesh filename="package://argos_description/meshes/RL_coxa_link_1.stl" scale="0.001 0.001 0.001"/>
     </geometry>
   </collision>
@@ -433,5 +453,5 @@
     <origin xyz="-0.176517 0.111383 -0.027133" rpy="0 0 0"/>
     <geometry>
-      <mesh filename="package://Argos_description/meshes/RL_femur_link_1.stl" scale="0.001 0.001 0.001"/>
+      <mesh filename="package://argos_description/meshes/RL_femur_link_1.stl" scale="0.001 0.001 0.001"/>
     </geometry>
     <material name="silver"/>
@@ -440,5 +460,5 @@
     <origin xyz="-0.176517 0.111383 -0.027133" rpy="0 0 0"/>
     <geometry>
-      <mesh filename="package://Argos_description/meshes/RL_femur_link_1.stl" scale="0.001 0.001 0.001"/>
+      <mesh filename="package://argos_description/meshes/RL_femur_link_1.stl" scale="0.001 0.001 0.001"/>
     </geometry>
   </collision>
@@ -453,5 +473,5 @@
     <origin xyz="-0.275538 0.110742 0.052389" rpy="0 0 0"/>
     <geometry>
-      <mesh filename="package://Argos_description/meshes/RL_tibia_link_1.stl" scale="0.001 0.001 0.001"/>
+      <mesh filename="package://argos_description/meshes/RL_tibia_link_1.stl" scale="0.001 0.001 0.001"/>
     </geometry>
     <material name="silver"/>
@@ -460,5 +480,5 @@
     <origin xyz="-0.275538 0.110742 0.052389" rpy="0 0 0"/>
     <geometry>
-      <mesh filename="package://Argos_description/meshes/RL_tibia_link_1.stl" scale="0.001 0.001 0.001"/>
+      <mesh filename="package://argos_description/meshes/RL_tibia_link_1.stl" scale="0.001 0.001 0.001"/>
     </geometry>
   </collision>
@@ -473,5 +493,5 @@
     <origin xyz="0.041083 0.111383 -0.027133" rpy="0 0 0"/>
     <geometry>
-      <mesh filename="package://Argos_description/meshes/FL_shoulder_link_1.stl" scale="0.001 0.001 0.001"/>
+      <mesh filename="package://argos_description/meshes/FL_shoulder_link_1.stl" scale="0.001 0.001 0.001"/>
     </geometry>
     <material name="silver"/>
@@ -480,5 +500,5 @@
     <origin xyz="0.041083 0.111383 -0.027133" rpy="0 0 0"/>
     <geometry>
-      <mesh filename="package://Argos_description/meshes/FL_shoulder_link_1.stl" scale="0.001 0.001 0.001"/>
+      <mesh filename="package://argos_description/meshes/FL_shoulder_link_1.stl" scale="0.001 0.001 0.001"/>
     </geometry>
   </collision>
@@ -493,5 +513,5 @@
     <origin xyz="0.085083 0.115383 -0.002716" rpy="0 0 0"/>
     <geometry>
-      <mesh filename="package://Argos_description/meshes/FL_30mm_linkage_1.stl" scale="0.001 0.001 0.001"/>
+      <mesh filename="package://argos_description/meshes/FL_30mm_linkage_1.stl" scale="0.001 0.001 0.001"/>
     </geometry>
     <material name="silver"/>
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