Commit message: Worked last night
switched to chase's microcontroller code

File: leg_controller/full_body_pose_dashboard/public/argos_description/urdf/Argos.urdf (robot description, URDF)
Before this commit: robot Argos, 39 links, 38 joints
Joints:
- joint FL_coxa_joint: limit lower=-0.524 upper=0.524 effort=4.41 velocity=6.28 -> (none); type revolute -> continuous
- joint FL_femur_joint: limit lower=-1.047 upper=2.094 effort=4.41 velocity=6.28 -> (none); type revolute -> continuous
- joint FL_tibia_joint: limit lower=-2.618 upper=0.0 effort=4.41 velocity=6.28 -> (none); type revolute -> continuous
- joint FR_coxa_joint: limit lower=-0.524 upper=0.524 effort=4.41 velocity=6.28 -> (none); type revolute -> continuous
- joint FR_femur_joint: limit lower=-1.047 upper=2.094 effort=4.41 velocity=6.28 -> (none); type revolute -> continuous
- joint FR_tibia_joint: limit lower=-2.618 upper=0.0 effort=4.41 velocity=6.28 -> (none); type revolute -> continuous
- joint RL_coxa_joint: limit lower=-0.524 upper=0.524 effort=4.41 velocity=6.28 -> (none); type revolute -> continuous
- joint RL_femur_joint: limit lower=-1.047 upper=2.094 effort=4.41 velocity=6.28 -> (none); type revolute -> continuous
- joint RL_tibia_joint: limit lower=-2.618 upper=0.0 effort=4.41 velocity=6.28 -> (none); type revolute -> continuous
- joint RR_coxa_joint: limit lower=-0.524 upper=0.524 effort=4.41 velocity=6.28 -> (none); type revolute -> continuous
- joint RR_femur_joint: limit lower=-1.047 upper=2.094 effort=4.41 velocity=6.28 -> (none); type revolute -> continuous
- joint RR_tibia_joint: limit lower=-2.618 upper=0.0 effort=4.41 velocity=6.28 -> (none); type revolute -> continuous
